File: rev1.f/POVSpinner.sch (KiCad schematic (older format))
At the start: 24 parts, among them P1 ISP, SW1 SW_RESET, SW2 SW_POWER, U1 Microchip_ATtiny85, X1 USBMICRO

Commit message: added new 5.3mm soic 8 footprint for AtTiny85
Parts:
- U1: footprint Housings_SOIC:SOIC-8_3.9x4.9mm_Pitch1.27mm -> Housings_SOIC:SOIJ-8_5.3x5.3mm_Pitch1.27mm
Changed lines of the file:
@@
 F 0 "U1" H 3700 2220 60  0000 C CNN
 F 1 "Microchip_ATtiny85" H 4700 3321 60  0000 C CNN
-F 2 "Housings_SOIC:SOIC-8_3.9x4.9mm_Pitch1.27mm" H 4100 3340 60  0001 C CNN
+F 2 "Housings_SOIC:SOIJ-8_5.3x5.3mm_Pitch1.27mm" H 4100 3340 60  0001 C CNN
 F 3 "" H 4100 3340 60  0001 C CNN
 	1    4100 3340
